Commit message: Imported upstream version '0.3.0' of 'upstream'

File: gazebo_oru/cititruck/cititruck_description/urdf/cititruck.xacro (robot description, xacro)
@@ -1,4 +1,14 @@
 <?xml version="1.0"?>
 <robot name="cititruck" xmlns:xacro="http://ros.org/wiki/xacro">
+    <xacro:arg name="tf_prefix" default="robot_xacro_default"/>
+    <xacro:arg name="velodyne" default="false"/>
+    <xacro:arg name="kinect2" default="false"/>
+    <xacro:arg name="kinect1" default="false"/> <!-- deprecated -->
+    <!-- Arguments used in cititruck.gazebo -->
+    <xacro:arg name="controller_prefix" default=""/>
+    <xacro:arg name="sensor_prefix" default=""/>
+    <xacro:arg name="sick_name" default="safety"/>
+    <xacro:arg name="ls2000_name" default="nav"/>
+    <xacro:arg name="kinect2_name" default=""/>
   <!-- Import all Gazebo-customization elements, including Gazebo colors -->
   <xacro:include filename="$(find cititruck_description)/urdf/cititruck.gazebo" />
@@ -304,4 +314,5 @@
       <joint name="kinect_joint" type="fixed">
 	<axis xyz="0 1 0" />
+ 	<!--origin xyz="0.5 0 0.7" rpy="${pi/2 + 0.5} 0 ${-pi/2}" /--> <!-- 0 2.5 0 -->
  	<origin xyz="0.5 0 0.7" rpy="0 2.5 0"/> <!-- 0 2.5 0 -->
 <!--  	<origin xyz="0.5 0 0.7" rpy="0 3.14159 0"/> -->
@@ -309,3 +320,10 @@
 	<child link="kinect_link"/>
       </joint>
+      <link name="kinect_rgb_optical_link"/>
+      <joint name="kinect_optical_joint" type="fixed">
+        <axis xyz="0 1 0" />
+        <origin xyz="0.0 0.0 0.0" rpy="${-pi/2} 0 ${-pi/2}"/>
+        <parent link="kinect_link"/>
+        <child link="kinect_rgb_optical_link"/>
+      </joint>
 </robot>

File: gazebo_oru/cititruck/cititruck_description/urdf/iliad_velodyne_cititruck.xacro (robot description, xacro)
@@ -5,4 +5,10 @@
     <xacro:arg name="kinect2" default="false"/>
     <xacro:arg name="kinect1" default="false"/> <!-- deprecated -->
+    <!-- Arguments used in cititruck.gazebo -->
+    <xacro:arg name="controller_prefix" default=""/>
+    <xacro:arg name="sensor_prefix" default=""/>
+    <xacro:arg name="sick_name" default="safety"/>
+    <xacro:arg name="ls2000_name" default="nav"/>
+    <xacro:arg name="kinect2_name" default=""/>
     <!-- Import all Gazebo-customization elements, including Gazebo colors -->
     <xacro:include filename="$(find cititruck_description)/urdf/cititruck.gazebo"/>
@@ -281,5 +287,5 @@
     <!-- SENSORS START HERE -->
     <!-- SICK laser -->
-    <link name="safety_laser_link">
+    <link name="$(arg sick_name)_link">
         <collision>
             <origin xyz="0 0 0" rpy="0 0 0"/>
@@ -300,12 +306,12 @@
         </inertial>
     </link>
-    <joint name="safety_laser_joint" type="fixed">
+    <joint name="$(arg sick_name)_joint" type="fixed">
         <axis xyz="0 1 0"/>
         <origin xyz="1.4 0 0.02" rpy="3.14159 0 0"/>
         <parent link="base_link"/>
-        <child link="safety_laser_link"/>
+        <child link="$(arg sick_name)_link"/>
     </joint>
     <!-- LS2000 navigation/localization laser -->
-    <link name="nav_laser_link">
+    <link name="$(arg ls2000_name)_link">
         <collision>
             <origin xyz="0 0 0" rpy="0 0 0"/>
@@ -326,13 +332,13 @@
         </inertial>
     </link>
-    <joint name="nav_laser_joint" type="fixed">
+    <joint name="$(arg ls2000_name)_joint" type="fixed">
         <origin xyz="0.8 0 0.85" rpy="0 0 0"/>
         <parent link="base_link"/>
-        <child link="nav_laser_link"/>
+        <child link="$(arg ls2000_name)_link"/>
     </joint>
     <!-- Velodyne VLP16 -->
     <xacro:if value="$(arg velodyne)">
       <xacro:include filename="$(find velodyne_description)/urdf/VLP-16.urdf.xacro"/>
-      <VLP-16 parent="base_link" prefix="$(arg tf_prefix)" name="velodyne" topic="/velodyne_points" hz="10" samples="440">
+      <VLP-16 parent="base_link" prefix="$(arg tf_prefix)/velodyne" name="velodyne" topic="/velodyne_points" hz="10" samples="440">
           <origin xyz="0.8 0 0.95" rpy="0 0 0" />
       </VLP-16>
